File: Hardware/Version2/F100_B200_Test_Bop_V2/F100_B200_Test_Bop_V2.kicad_pcb (KiCad board)
At the start: 2 copper layers, 180 x 120 mm, 67 parts, among them IC1 OPA548T, J1 Screw_Terminal_01x08, J10 ESQ-108-14-T-S, J11 ESQ-108-14-T-S, J12 ESQ-110-14-T-S, J13 ESQ-108-14-T-S, J14 TB001-500-10BE, J15 Screw_Terminal_01x08, J16 102-TBL004V-508-18BE-2GY-ND, J17 ESQ-118-14-G-D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

Commit message: clean up
Connections:
- IC1 pad 6: Net-(IC1-Pad6) -> /BatSimulator
- R12 pad 1: Net-(IC1-Pad6) -> /BatSimulator
- U6 pad IN+: Net-(IC1-Pad6) -> /Charger
- U6 pad IN-: Net-(U6-PadIN-) -> /BatSimulator
Routing:
- net /BatSimulator: track 0.00 -> 76.3 mm
- net Net-(IC1-Pad6): track 70.7 -> 0.00 mm

Commit message: added mechanical dwgs
Parts:
- added D17: 1N4004-TP, Diode_THT:D_DO-41_SOD81_P10.16mm_Horizontal, F.Cu at (115.7, 16.9)
- added D18: 1N4004-TP, Diode_THT:D_DO-41_SOD81_P10.16mm_Horizontal, F.Cu at (125.9, 16.9)
- added D19: D_Zener, Diode_THT:D_DO-35_SOD27_P7.62mm_Horizontal, F.Cu at (114.3, 45.7)
- added D20: D_Zener, Diode_THT:D_DO-35_SOD27_P7.62mm_Horizontal, F.Cu at (117.0, 45.6)
- added Q6: Q_NPN_EBC, Package_TO_SOT_THT:TO-92L_Inline_Wide, F.Cu at (111.8, 24.6)
- added Q7: Q_NPN_EBC, Package_TO_SOT_THT:TO-92L_Inline_Wide, F.Cu at (122.0, 24.3)
- added R22: 2.7k, Resistor_THT:R_Axial_DIN0204_L3.6mm_D1.6mm_P7.62mm_Horizontal, F.Cu at (119.5, 31.2)
- added R23: 2.7k, Resistor_THT:R_Axial_DIN0204_L3.6mm_D1.6mm_P7.62mm_Horizontal, F.Cu at (122.0, 31.1)
- added R24: 10k, Resistor_THT:R_Axial_DIN0204_L3.6mm_D1.6mm_P7.62mm_Horizontal, F.Cu at (101.0, 16.5)
- added R25: 10k, Resistor_THT:R_Axial_DIN0204_L3.6mm_D1.6mm_P7.62mm_Horizontal, F.Cu at (104.4, 16.6)
- moved Q5 24.7 mm to (141.6, 24.0)
- moved D16 24.6 mm to (145.3, 16.5)
- moved D15 22.6 mm to (135.5, 16.6)
- moved Q4 22.4 mm to (131.8, 24.4)
- moved R18 22.0 mm to (127.1, 31.1)
- moved R17 22.0 mm to (124.5, 31.1)
- moved Q2 19.5 mm to (151.6, 23.9)
- moved D13 19.3 mm to (155.3, 16.5)
- moved D14 17.7 mm to (164.9, 16.4)
- moved Q3 17.7 mm to (161.2, 24.0)
- moved R20 0.13 mm to (136.1, 31.0)
- moved R21 0.08 mm to (138.6, 31.0)
Connections:
- J14 pad 10: /D8 -> Net-(D16-Pad1)
- J14 pad 5: /D13 -> Net-(J14-Pad5)
- J14 pad 6: /D12 -> Net-(J14-Pad6)
- J14 pad 7: /D11 -> Net-(D17-Pad1)
- J14 pad 8: /D10 -> Net-(D18-Pad1)
- J14 pad 9: /D9 -> Net-(D15-Pad1)
- J5 pad 7: Net-(D15-Pad1) -> /D1
- J5 pad 8: Net-(D16-Pad1) -> /D0
- J7 pad 1: /12VDC -> /BatSimulator
- R17 pad 2: /D1 -> /D9
- R18 pad 2: /D0 -> /D8
- U6 pad IN-: /BatSimulator -> Net-(U6-PadIN-)
Routing:
- net /D1: track 4.35 -> 62.6 mm
- net /D0: track 4.40 -> 58.6 mm
- net /BatSimulator: track 76.3 -> 39.0 mm
- net /D10: track 38.5 -> 4.11 mm
- net /D9: track 37.4 -> 4.09 mm
- net /D8: track 36.4 -> 4.08 mm
- net /D11: track 105.0 -> 81.0 mm
- net Net-(D18-Pad1): track 0.00 -> 19.7 mm
- net Net-(D17-Pad1): track 0.00 -> 16.9 mm
- net Net-(D13-Pad1): track 31.7 -> 15.4 mm
- net /D13: track 41.5 -> 27.1 mm
- net /D12: track 40.5 -> 26.6 mm
- net Net-(Q3-Pad2): track 9.24 -> 23.1 mm
- net Net-(Q6-Pad2): track 0.00 -> 13.1 mm
- net Net-(D16-Pad1): track 15.8 -> 26.7 mm
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