File: Hardware/Version2/F100_B200_Test_Bop_V2/F100_B200_Test_Bop_V2.sch (KiCad schematic (older format))
At the start: 67 parts, among them IC1 OPA548T, J1 Screw_Terminal_01x08, J10 ESQ-108-14-T-S, J11 ESQ-108-14-T-S, J12 ESQ-110-14-T-S, J13 ESQ-108-14-T-S, J14 TB001-500-10BE, J15 Screw_Terminal_01x08, J16 102-TBL004V-508-18BE-2GY-ND, J17 ESQ-118-14-G-D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

Commit message: "change voltage control to PID"
Parts:
- added J4: Screw_Terminal_01x04, lib_fp_pretty:CUI_TB001-500-04BE, symbol Connector:Screw_Terminal_01x04
Connections:
- net BatSimulator: now reaches IC1.6 (OUT), R12.1
- net BatSimulator: now also J4.1 (Pin_1); no longer U6.IN+ (7)
- net Charger: now reaches U6.IN- (8)
- net Charger: now also J4.3 (Pin_3)
- new net In+: J4.2 (Pin_2), U6.IN+ (7)
Other:
- note added: "Plus_load"
- note added: "Power_On_Not"
- note added: "STAT_1"
- note added: "STAT_2"
- moved on the sheet: U6
Changed lines of the file:
@@
 	1    0    0    -1
 $EndComp
-$Comp
-L F100_B200_Test_Bop_V2-rescue:INA260-F100B200TestPanel U6
-U 1 1 5F8A9991
-P 4050 1950
-F 0 "U6" H 4000 2325 50  0000 C CNN
-F 1 "INA260" H 4000 2234 50  0000 C CNN
-F 2 "lib_fp_pretty:Adafruit_INA260" H 4050 1950 50  0001 C CNN
-F 3 "https://cdn-learn.adafruit.com/downloads/pdf/adafruit-ina260-current-voltage-power-sensor-breakout.pdf" H 4050 1950 50  0001 C CNN
-F 4 "INA260 Current Monitor Power Management Evaluation Board" H 4050 1950 50  0001 C CNN "Description"
-F 5 "1528-2955-ND" H 4050 1950 50  0001 C CNN "DigikeyPart#"
-	1    4050 1950
-	-1   0    0    -1
-$EndComp
-Wire Wire Line
-	3000 1950 3650 1950
-Connection ~ 3000 1950
 Wire Wire Line
 	1500 950  1700 950
@@
 Wire Wire Line
 	900  2200 1150 2200
-Wire Wire Line
-	4550 1900 4850 1900
 $Comp
 L Connector:Screw_Terminal_01x02 J6
@@
 Text Label 750  1850 2    50   ~ 0
 D20
-Text Label 4550 1800 0    50   ~ 0
-+3V3
 $Comp
 L power:GND #PWR021
 U 1 1 5FB96DDE
-P 4850 1900
-F 0 "#PWR021" H 4850 1650 50  0001 C CNN
-F 1 "GND" H 4855 1727 50  0000 C CNN
-F 2 "" H 4850 1900 50  0001 C CNN
-F 3 "" H 4850 1900 50  0001 C CNN
-	1    4850 1900
-	0    -1   -1   0
-$EndComp
-Text Label 4550 2000 0    50   ~ 0
-D21
-Text Label 4550 2100 0    50   ~ 0
-D20
+P 4575 2650
+F 0 "#PWR021" H 4575 2400 50  0001 C CNN
+F 1 "GND" H 4580 2477 50  0000 C CNN
+F 2 "" H 4575 2650 50  0001 C CNN
+F 3 "" H 4575 2650 50  0001 C CNN
+	1    4575 2650
+	0    -1   -1   0
+$EndComp
 Text Label 1150 700  0    50   ~ 0
 +3V3
@@
 Text Label 3150 1000 0    50   ~ 0
 12VDC
+Text Label 3000 1950 0    50   ~ 0
+BatSimulator
+Text Label 4275 2850 0    50   ~ 0
+D20
+Text Label 4275 2750 0    50   ~ 0
+D21
+Text Label 4275 2550 0    50   ~ 0
++3V3
+Wire Wire Line
+	4275 2650 4575 2650
+$Comp
+L F100_B200_Test_Bop_V2-rescue:INA260-F100B200TestPanel U6
+U 1 1 5F8A9991
+P 3775 2700
+F 0 "U6" H 3725 3075 50  0000 C CNN
+F 1 "INA260" H 3725 2984 50  0000 C CNN
+F 2 "lib_fp_pretty:Adafruit_INA260" H 3775 2700 50  0001 C CNN
+F 3 "https://cdn-learn.adafruit.com/downloads/pdf/adafruit-ina260-current-voltage-power-sensor-breakout.pdf" H 3775 2700 50  0001 C CNN
+F 4 "INA260 Current Monitor Power Management Evaluation Board" H 3775 2700 50  0001 C CNN "Description"
+F 5 "1528-2955-ND" H 3775 2700 50  0001 C CNN "DigikeyPart#"
+	1    3775 2700
+	-1   0    0    -1
+$EndComp
+$Comp
+L Connector:Screw_Terminal_01x04 J4
+U 1 1 5FDE24B8
+P 4025 950
+F 0 "J4" H 4105 896 50  0000 L CNN
+F 1 "Screw_Terminal_01x04" H 4105 851 50  0001 L CNN
+F 2 "lib_fp_pretty:CUI_TB001-500-04BE" H 4025 950 50  0001 C CNN
+F 3 "https://www.cuidevices.com/product/resource/digikeypdf/tb001-500.pdf" H 4025 950 50  0001 C CNN
+F 4 "4 Position Wire to Board Terminal Block Horizontal with Board 0.197\" (5.00mm) Through Hole" H 4025 950 50  0001 C CNN "Description"
+F 5 "102-6136-ND" H 4025 950 50  0001 C CNN "DigikeyPart#"
+	1    4025 950
+	0    -1   -1   0
+$EndComp
+Text Label 3375 2700 2    50   ~ 0
+In+
+Text Label 3375 2800 2    50   ~ 0
+Charger
+Text Label 3925 1150 3    50   ~ 0
+BatSimulator
+Text Label 4025 1150 3    50   ~ 0
+In+
+Text Label 4125 1150 3    50   ~ 0
+Charger
+Text Notes 10250 2825 0    50   ~ 0
+STAT_1
+Text Notes 10250 2925 0    50   ~ 0
+STAT_2
+Text Notes 10250 3025 0    50   ~ 0
+Power_On_Not
+Text Notes 10250 3125 0    50   ~ 0
+Plus_load
 $EndSCHEMATC

Commit message: clean up
Parts:
- removed J4: Screw_Terminal_01x04, lib_fp_pretty:CUI_TB001-500-04BE, symbol Connector:Screw_Terminal_01x04
Connections:
- net In+ is gone; now on net Charger: U6.IN+ (7)
- net BatSimulator: now also U6.IN- (8)
- net Charger: no longer U6.IN- (8)
Changed lines of the file:
@@
 	-1   0    0    -1
 $EndComp
-$Comp
-L Connector:Screw_Terminal_01x04 J4
-U 1 1 5FDE24B8
-P 4025 950
-F 0 "J4" H 4105 896 50  0000 L CNN
-F 1 "Screw_Terminal_01x04" H 4105 851 50  0001 L CNN
-F 2 "lib_fp_pretty:CUI_TB001-500-04BE" H 4025 950 50  0001 C CNN
-F 3 "https://www.cuidevices.com/product/resource/digikeypdf/tb001-500.pdf" H 4025 950 50  0001 C CNN
-F 4 "4 Position Wire to Board Terminal Block Horizontal with Board 0.197\" (5.00mm) Through Hole" H 4025 950 50  0001 C CNN "Description"
-F 5 "102-6136-ND" H 4025 950 50  0001 C CNN "DigikeyPart#"
-	1    4025 950
-	0    -1   -1   0
-$EndComp
-Text Label 3375 2700 2    50   ~ 0
-In+
-Text Label 3375 2800 2    50   ~ 0
-Charger
-Text Label 3925 1150 3    50   ~ 0
-BatSimulator
-Text Label 4025 1150 3    50   ~ 0
-In+
-Text Label 4125 1150 3    50   ~ 0
+Text Label 3325 2500 1    50   ~ 0
 Charger
 Text Notes 10250 2825 0    50   ~ 0
@@
 Text Notes 10250 3125 0    50   ~ 0
 Plus_load
+Wire Wire Line
+	3000 1950 3225 1950
+Wire Wire Line
+	3225 1950 3225 2800
+Wire Wire Line
+	3225 2800 3375 2800
+Connection ~ 3000 1950
+Wire Wire Line
+	3375 2700 3325 2700
+Wire Wire Line
+	3325 2700 3325 2500
 $EndSCHEMATC

Commit message: added mechanical dwgs
Parts:
- added D17, D18: 1N4004-TP, Diode_THT:D_DO-41_SOD81_P10.16mm_Horizontal, symbol Device:D
- added D19, D20: D_Zener, Diode_THT:D_DO-35_SOD27_P7.62mm_Horizontal, symbol Device:D_Zener
- added Q6, Q7: Q_NPN_EBC, Package_TO_SOT_THT:TO-92L_Inline_Wide, symbol Device:Q_NPN_EBC
- added R22, R23: 2.7k, Resistor_THT:R_Axial_DIN0204_L3.6mm_D1.6mm_P7.62mm_Horizontal, symbol Device:R
- added R24, R25: 10k, Resistor_THT:R_Axial_DIN0204_L3.6mm_D1.6mm_P7.62mm_Horizontal, symbol Device:R
- J10, J11, J13, J8, J9: DigikeyPart# (none) -> SAM9303-ND
Connections:
- net 12VDC: no longer J7.1 (Pin_1)
- net BatSimulator: now also J7.1 (Pin_1); no longer U6.IN- (8)
- net D0: now also J5.8 (Pin_8); no longer R18.2
- net D1: now also J5.7 (Pin_7); no longer R17.2
- net D10: now also R23.2; no longer J14.8 (Pin_8)
- net D11: now also R22.2; no longer J14.7 (Pin_7)
- net D12: now also D20.1 (K), R25.2; no longer J14.6 (Pin_6)
- net D13: now also D19.1 (K), R24.2; no longer J14.5 (Pin_5)
- net D8: now also R18.2; no longer J14.10 (Pin_10)
- net D9: now also R17.2; no longer J14.9 (Pin_9)
- net GND: now also D17.2 (A), D18.2 (A), D19.2 (A), D20.2 (A), Q6.1 (E), Q7.1 (E)
- net at D15.1 (K), Q4.3 (C): now also J14.9 (Pin_9); no longer J5.7 (Pin_7)
- net at D16.1 (K), Q5.3 (C): now also J14.10 (Pin_10); no longer J5.8 (Pin_8)
- new net: J14.5 (Pin_5), R24.1
- new net: J14.6 (Pin_6), R25.1
- new net: D17.1 (K), J14.7 (Pin_7), Q6.3 (C)
- new net: D18.1 (K), J14.8 (Pin_8), Q7.3 (C)
- new net: Q7.2 (B), R23.1
- new net: Q6.2 (B), R22.1
Other:
- note removed: "External/Internal Select"
- moved on the sheet: D10, D11, D12, D13, D14, D15, D16, D9, HS2, J11, J12, J13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
